Commit message: rename husky_description --> husky_ur_description, use HUSKY_URDF_EXTRAS rather than HUSKY_DESCRIPTION in env-hook.

File: husky_ur_description/urdf/accessories/husky_ur_accessories.urdf.xacro (robot description, xacro)
@@ -5,5 +5,5 @@
   <xacro:include filename="$(find robotiq_c_model_viz)/urdf/c_model_open.urdf.xacro" />
   <!-- RealSense D41X Camera -->
-  <xacro:include filename="$(find husky_description)/urdf/accessories/realsense_d410.urdf.xacro"/>
+  <xacro:include filename="$(find husky_ur_description)/urdf/accessories/realsense_d410.urdf.xacro"/>
   <!-- CHANGE BELOW VALUES DURING INTEGRATION -->
   <!-- MUST CHANGE TO UR5, UR3 or UR10 depending on needs -->
@@ -62,10 +62,10 @@
     <visual>
       <geometry>
-        <mesh filename="package://husky_description/meshes/integration_arch.dae" />
+        <mesh filename="package://husky_ur_description/meshes/integration_arch.dae" />
       </geometry>
     </visual>
     <collision>
       <geometry>
-        <mesh filename="package://husky_description/meshes/integration_arch.dae" />
+        <mesh filename="package://husky_ur_description/meshes/integration_arch.dae" />
       </geometry>
     </collision>

File: husky_ur_description/urdf/accessories/kinect_camera.urdf.xacro (robot description, xacro)
@@ -34,5 +34,5 @@
         <origin xyz="0 0 0" rpy="0 0 ${M_PI/2}"/>
         <geometry>
-          <mesh filename="package://husky_description/meshes/accessories/kinect.dae" />
+          <mesh filename="package://husky_ur_description/meshes/accessories/kinect.dae" />
         </geometry>
       </visual>

File: husky_ur_description/urdf/accessories/realsense_d410.urdf.xacro (robot description, xacro)
@@ -41,5 +41,5 @@
         <origin xyz="0.0 0.0 0.0" rpy="1.5708 0.0 1.5708"/>
         <geometry>
-          <mesh filename="package://husky_description/meshes/realsense_d415.dae" />
+          <mesh filename="package://husky_ur_description/meshes/realsense_d415.dae" />
         </geometry>
       </visual>

File: husky_ur_description/urdf/accessories/sensor_arch.urdf.xacro (robot description, xacro)
@@ -7,5 +7,5 @@
              <visual>
                  <geometry>
-                     <mesh filename="package://husky_description/meshes/accessories/${size}_mm_sensor_arch.dae" />
+                     <mesh filename="package://husky_ur_description/meshes/accessories/${size}_mm_sensor_arch.dae" />
                  </geometry>
              </visual>
@@ -13,5 +13,5 @@
                  <origin xyz="0 0 0" rpy="0 0 0"/>
                  <geometry>
-                     <mesh filename="package://husky_description/meshes/accessories/${size}_mm_sensor_arch.dae" />
+                     <mesh filename="package://husky_ur_description/meshes/accessories/${size}_mm_sensor_arch.dae" />
                  </geometry>
              </collision>

File: husky_ur_description/urdf/accessories/sick_lms1xx_mount.urdf.xacro (robot description, xacro)
@@ -34,5 +34,5 @@
         <geometry>
           <!-- Origin of this mesh is the base of the bracket. -->
-          <mesh filename="package://husky_description/meshes/accessories/lms1xx_mount.dae" />
+          <mesh filename="package://husky_ur_description/meshes/accessories/lms1xx_mount.dae" />
         </geometry>
       </visual>

File: husky_ur_description/urdf/decorations.urdf.xacro (robot description, xacro)
@@ -28,5 +28,5 @@
         <origin xyz="0 0 0" rpy="0 0 0" />
         <geometry>
-          <mesh filename="package://husky_description/meshes/top_chassis.dae" />
+          <mesh filename="package://husky_ur_description/meshes/top_chassis.dae" />
         </geometry>
       </visual>
@@ -41,5 +41,5 @@
       <visual>
         <geometry>
-          <mesh filename="package://husky_description/meshes/user_rail.dae" />
+          <mesh filename="package://husky_ur_description/meshes/user_rail.dae" />
         </geometry>
       </visual>
@@ -55,5 +55,5 @@
       <visual>
         <geometry>
-          <mesh filename="package://husky_description/meshes/bumper.dae" />
+          <mesh filename="package://husky_ur_description/meshes/bumper.dae" />
         </geometry>
       </visual>
@@ -69,5 +69,5 @@
       <visual>
         <geometry>
-          <mesh filename="package://husky_description/meshes/bumper.dae" />
+          <mesh filename="package://husky_ur_description/meshes/bumper.dae" />
         </geometry>
       </visual>
@@ -85,5 +85,5 @@
           <origin xyz="0 0 0" rpy="0 0 0" />
           <geometry>
-            <mesh filename="package://husky_description/meshes/top_plate.dae" />
+            <mesh filename="package://husky_ur_description/meshes/top_plate.dae" />
           </geometry>
         </visual>
@@ -91,5 +91,5 @@
           <origin xyz="0 0 0" rpy="0 0 0"/>
           <geometry>
-            <mesh filename="package://husky_description/meshes/top_plate.dae" />
+            <mesh filename="package://husky_ur_description/meshes/top_plate.dae" />
           </geometry>
         </collision>

File: husky_ur_description/urdf/description.xacro (robot description, xacro)
@@ -24,5 +24,5 @@
   <xacro:arg name="laser_enabled" default="false" />
   <xacro:arg name="kinect_enabled" default="false" />
-  <xacro:include filename="$(find husky_description)/urdf/husky.urdf.xacro" />
+  <xacro:include filename="$(find husky_ur_description)/urdf/husky.urdf.xacro" />
   <xacro:husky_robot />
 </robot>

File: husky_ur_description/urdf/husky.urdf.xacro (robot description, xacro)
@@ -23,10 +23,10 @@
 <robot name="husky_robot" xmlns:xacro="http://ros.org/wiki/xacro">
   <!-- Included URDF/XACRO Files -->
-  <xacro:include filename="$(find husky_description)/urdf/decorations.urdf.xacro" />
-  <xacro:include filename="$(find husky_description)/urdf/wheel.urdf.xacro" />
-  <xacro:include filename="$(find husky_description)/urdf/accessories/kinect_camera.urdf.xacro"/>
-  <xacro:include filename="$(find husky_description)/urdf/accessories/sick_lms1xx_mount.urdf.xacro"/>
-  <xacro:include filename="$(find husky_description)/urdf/accessories/sensor_arch.urdf.xacro"/>
-  <xacro:include filename="$(find husky_description)/urdf/accessories/husky_ur_accessories.urdf.xacro"/>
+  <xacro:include filename="$(find husky_ur_description)/urdf/decorations.urdf.xacro" />
+  <xacro:include filename="$(find husky_ur_description)/urdf/wheel.urdf.xacro" />
+  <xacro:include filename="$(find husky_ur_description)/urdf/accessories/kinect_camera.urdf.xacro"/>
+  <xacro:include filename="$(find husky_ur_description)/urdf/accessories/sick_lms1xx_mount.urdf.xacro"/>
+  <xacro:include filename="$(find husky_ur_description)/urdf/accessories/sensor_arch.urdf.xacro"/>
+  <xacro:include filename="$(find husky_ur_description)/urdf/accessories/husky_ur_accessories.urdf.xacro"/>
   <property name="M_PI" value="3.14159"/>
   <!-- Base Size -->
@@ -47,5 +47,5 @@
         <origin xyz="0 0 0" rpy="0 0 0" />
         <geometry>
-          <mesh filename="package://husky_description/meshes/base_link.dae" />
+          <mesh filename="package://husky_ur_description/meshes/base_link.dae" />
         </geometry>
       </visual>

File: husky_ur_description/urdf/wheel.urdf.xacro (robot description, xacro)
@@ -32,5 +32,5 @@
 				<origin xyz="0 0 0" rpy="0 0 0" />
 				<geometry>
-					<mesh filename="package://husky_description/meshes/wheel.dae" />
+					<mesh filename="package://husky_ur_description/meshes/wheel.dae" />
 				</geometry>
 			</visual>
